File: lis3dh_board.kicad_sch (KiCad schematic)
At the start: 23 parts, among them J1 T4_IF, J2 BQ25798_BOARD, J3 WL-125, Q1 BSS138, U1 TLV75530PDBV, U2 LIS3DH

Commit message: Add PicoBlade connector for the RFID antenna coil
The 125kHz antenna coil now plugs into J4 (Molex PicoBlade 53047-0210,
1.25mm 2-pin) and is routed to the WL-125 ANT1/ANT2 pins (J3 pins 2-3)
instead of being soldered to the module. Layout notes cover the
~100Vpp on these traces.

Co-Authored-By: Claude Opus 5.5 <noreply@anthropic.com>
Claude-Session: https://claude.ai/code/session_012K15v8QNdkAoa4NiCNiWuG
Parts:
- added J4: RFID_ANT, Connector_Molex:Molex_PicoBlade_53047-0210_1x02_P1.25mm_Vertical, symbol Connector_Generic:Conn_01x02
Connections:
- net ANT1: now reaches J3.2 (Pin_2)
- net ANT1: now also J4.1 (Pin_1)
- net ANT2: now reaches J3.3 (Pin_3)
- net ANT2: now also J4.2 (Pin_2)
- no-connect marks 9 -> 7
Other:
- note added: "J3 -> WL-125 RFID (1x10 socket, 2.54mm) J3 pin = module pin + 1 1: key (next to module pin 1), NC 2,3: ANT1/2 -> J4 antenna connector, ~100Vpp 4: ASCII select = VCC_RF (UART mode) 5: BEEP (NC) 6: TX 9600 8N1, 5V -> Q1 level shifter -> RFID_TX 3.0V 7: Wiegand D0 (NC) 8: /RESET (R7 pull-up) 9: GND 10: VCC_RF (5V, 3-stage RC filtered)"
- note added: "J4 -> RFID antenna coil (Molex PicoBlade 1.25mm, 2-pin) ANT1/ANT2 carry ~50-100Vpp at 125kHz: short, parallel traces; >=0.5mm clearance; no copper pour around them"
- note removed: "J3 -> WL-125 RFID (1x10 socket, 2.54mm) J3 pin = module pin + 1 1: key (next to module pin 1), NC 2,3: ANT1/2 - coil soldered on module, ~100Vpp, NC here 4: ASCII select = VCC_RF (UART mode) 5: BEEP (NC) 6: TX 9600 8N1, 5V -> Q1 level shifter -> RFID_TX 3.0V 7: Wiegand D0 (NC) 8: /RESET (R7 pull-up) 9: GND 10: VCC_RF (5V, 3-stage RC filtered)"
Changed lines of the file:
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@@
   )
   (no_connect (at 223.52 134.62))
-  (no_connect (at 223.52 137.16))
-  (no_connect (at 223.52 139.7))
+  (wire (pts (xy 223.52 137.16) (xy 220.98 137.16))
+    (stroke (width 0) (type default))
+  )
+  (label "ANT1" (at 220.98 137.16 180) (fields_autoplaced)
+    (effects (font (size 1.27 1.27)) (justify right bottom))
+  )
+  (wire (pts (xy 223.52 139.7) (xy 220.98 139.7))
+    (stroke (width 0) (type default))
+  )
+  (label "ANT2" (at 220.98 139.7 180) (fields_autoplaced)
+    (effects (font (size 1.27 1.27)) (justify right bottom))
+  )
   (wire (pts (xy 223.52 142.24) (xy 220.98 142.24))
     (stroke (width 0) (type default))
@@
     (effects (font (size 1.27 1.27)) (justify right bottom))
   )
-  (text "J3 -> WL-125 RFID (1x10 socket, 2.54mm)\nJ3 pin = module pin + 1\n1: key (next to module pin 1), NC\n2,3: ANT1/2 - coil soldered on module, ~100Vpp, NC here\n4: ASCII select = VCC_RF (UART mode)\n5: BEEP (NC)\n6: TX 9600 8N1, 5V -> Q1 level shifter -> RFID_TX 3.0V\n7: Wiegand D0 (NC)\n8: /RESET (R7 pull-up)\n9: GND\n10: VCC_RF (5V, 3-stage RC filtered)" (at 213.36 106.68 0)
+  (text "J3 -> WL-125 RFID (1x10 socket, 2.54mm)\nJ3 pin = module pin + 1\n1: key (next to module pin 1), NC\n2,3: ANT1/2 -> J4 antenna connector, ~100Vpp\n4: ASCII select = VCC_RF (UART mode)\n5: BEEP (NC)\n6: TX 9600 8N1, 5V -> Q1 level shifter -> RFID_TX 3.0V\n7: Wiegand D0 (NC)\n8: /RESET (R7 pull-up)\n9: GND\n10: VCC_RF (5V, 3-stage RC filtered)" (at 213.36 106.68 0)
     (effects (font (size 1.27 1.27)) (justify left bottom))
   )
+  (symbol (lib_id "Connector_Generic:Conn_01x02") (at 228.6 172.72 0) (unit 1)
+    (in_bom yes) (on_board yes) (dnp no)
+    (property "Reference" "J4" (at 232.41 171.45 0)
+      (effects (font (size 1.27 1.27)) (justify left))
+    )
+    (property "Value" "RFID_ANT" (at 232.41 173.99 0)
+      (effects (font (size 1.27 1.27)) (justify left))
+    )
+    (property "Footprint" "Connector_Molex:Molex_PicoBlade_53047-0210_1x02_P1.25mm_Vertical" (at 228.6 172.72 0)
+      (effects (font (size 1.27 1.27)) hide)
+    )
+    (property "Datasheet" "~" (at 228.6 172.72 0)
+      (effects (font (size 1.27 1.27)) hide)
+    )
+    (property "MPN" "Molex 53047-0210" (at 228.6 172.72 0)
+      (effects (font (size 1.27 1.27)) hide)
+    )
+    (pin "1")
+    (pin "2")
+    (instances
+      (project "lis3dh_board"
+        (path "/1b8e18d0-3822-5ef2-b7bb-caef133ff686" (reference "J4") (unit 1))
+      )
+    )
+  )
+  (wire (pts (xy 223.52 172.72) (xy 220.98 172.72))
+    (stroke (width 0) (type default))
+  )
+  (label "ANT1" (at 220.98 172.72 180) (fields_autoplaced)
+    (effects (font (size 1.27 1.27)) (justify right bottom))
+  )
+  (wire (pts (xy 223.52 175.26) (xy 220.98 175.26))
+    (stroke (width 0) (type default))
+  )
+  (label "ANT2" (at 220.98 175.26 180) (fields_autoplaced)
+    (effects (font (size 1.27 1.27)) (justify right bottom))
+  )
+  (text "J4 -> RFID antenna coil (Molex PicoBlade 1.25mm, 2-pin)\nANT1/ANT2 carry ~50-100Vpp at 125kHz:\nshort, parallel traces; >=0.5mm clearance; no copper pour around them" (at 213.36 182.88 0)
+    (effects (font (size 1.27 1.27)) (justify left bottom))
+  )

Commit message: Add two M3 mounting holes
H1/H2 use MountingHole_3.2mm_M3 (non-plated) and are excluded from the
BOM. Placement is left for layout, near the accelerometer.

Co-Authored-By: Claude Opus 5.5 <noreply@anthropic.com>
Claude-Session: https://claude.ai/code/session_012K15v8QNdkAoa4NiCNiWuG
Parts:
- added H1, H2: M3, MountingHole:MountingHole_3.2mm_M3, symbol Mechanical:MountingHole
Other:
- note added: "H1/H2: M3 mounting holes (3.2mm, NPTH) mount near U2 so the accelerometer is held rigidly"
Changed lines of the file:
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@@
+    (effects (font (size 1.27 1.27)) (justify left bottom))
+  )
+  (symbol (lib_id "Mechanical:MountingHole") (at 40.64 228.6 0) (unit 1)
+    (in_bom no) (on_board yes) (dnp no)
+    (property "Reference" "H1" (at 40.64 222.6 0)
+      (effects (font (size 1.27 1.27)))
+    )
+    (property "Value" "M3" (at 40.64 235.6 0)
+      (effects (font (size 1.27 1.27)))
+    )
+    (property "Footprint" "MountingHole:MountingHole_3.2mm_M3" (at 40.64 228.6 0)
+      (effects (font (size 1.27 1.27)) hide)
+    )
+    (property "Datasheet" "~" (at 40.64 228.6 0)
+      (effects (font (size 1.27 1.27)) hide)
+    )
+    (instances
+      (project "lis3dh_board"
+        (path "/1b8e18d0-3822-5ef2-b7bb-caef133ff686" (reference "H1") (unit 1))
+      )
+    )
+  )
+  (symbol (lib_id "Mechanical:MountingHole") (at 55.88 228.6 0) (unit 1)
+    (in_bom no) (on_board yes) (dnp no)
+    (property "Reference" "H2" (at 55.88 222.6 0)
+      (effects (font (size 1.27 1.27)))
+    )
+    (property "Value" "M3" (at 55.88 235.6 0)
+      (effects (font (size 1.27 1.27)))
+    )
+    (property "Footprint" "MountingHole:MountingHole_3.2mm_M3" (at 55.88 228.6 0)
+      (effects (font (size 1.27 1.27)) hide)
+    )
+    (property "Datasheet" "~" (at 55.88 228.6 0)
+      (effects (font (size 1.27 1.27)) hide)
+    )
+    (instances
+      (project "lis3dh_board"
+        (path "/1b8e18d0-3822-5ef2-b7bb-caef133ff686" (reference "H2") (unit 1))
+      )
+    )
+  )
+  (text "H1/H2: M3 mounting holes (3.2mm, NPTH)\nmount near U2 so the accelerometer is held rigidly" (at 30.48 243.84 0)
     (effects (font (size 1.27 1.27)) (justify left bottom))
   )
