File: lis3dh_board.kicad_sch (KiCad schematic)
At the start: 26 parts, among them J1 T4_IF, J2 BQ25798_BOARD, J3 WL-125, J4 RFID_ANT, Q1 BSS138, U1 TLV75530PDBV, U2 LIS3DH

Commit message: Route the PCB and remove R3
- Remove R3 (CHG_INT pull-up); the pull-up lives on the charger board.
- Route the user's placement with Freerouting: netclasses Default
  (0.25mm), Power (+5V/VRF1/VRF2/VCC_RF, 0.4mm) and ANT (0.3mm, 0.4mm
  clearance), B.Cu GND plane, F.Cu GND pour plus 6 stitching vias.
  KiCad 10 DRC: no errors, 0 unconnected, schematic parity clean.
- Export Gerbers, drill and position files; add scripts/route.sh and
  route_pcb.py for re-routing; drop the obsolete gen_pcb.py.

Co-Authored-By: Claude Opus 5.5 <noreply@anthropic.com>
Claude-Session: https://claude.ai/code/session_012K15v8QNdkAoa4NiCNiWuG
Parts:
- removed C6: 100nF, Capacitor_SMD:C_0603_1608Metric, symbol Device:C
- removed H1: M3, MountingHole:MountingHole_3.2mm_M3, symbol Mechanical:MountingHole
- removed R3, R5: 10k, Resistor_SMD:R_0603_1608Metric, symbol Device:R
- removed R8, R9: 1R, Resistor_SMD:R_0805_2012Metric, symbol Device:R
- added C4: 10uF, Capacitor_SMD:C_0603_1608Metric, symbol Device:C
- added C7, C8: 1000uF 10V, Capacitor_SMD:CP_Elec_8x10.5, symbol Device:C_Polarized
- added J4: RFID_ANT, Connector_Molex:Molex_PicoBlade_53047-0210_1x02_P1.25mm_Vertical, symbol Connector_Generic:Conn_01x02
- added R6: 4.7R, Resistor_SMD:R_0805_2012Metric, symbol Device:R
- C5: renamed from R6; value 4.7R -> 1000uF 10V; footprint Resistor_SMD:R_0805_2012Metric -> Capacitor_SMD:CP_Elec_8x10.5; symbol Device:R -> Device:C_Polarized; LCSC (none) -> C278408; MPN (none) -> Panasonic EEE-FT1A102AP
- C6: renamed from C8; value 1000uF 10V -> 100nF; footprint Capacitor_SMD:CP_Elec_8x10.5 -> Capacitor_SMD:C_0603_1608Metric; symbol Device:C_Polarized -> Device:C; LCSC C278408 -> (none); MPN Panasonic EEE-FT1A102AP -> (none)
- H1: renamed from C4; value 10uF -> M3; footprint Capacitor_SMD:C_0603_1608Metric -> MountingHole:MountingHole_3.2mm_M3; symbol Device:C -> Mechanical:MountingHole; now left out of the parts list
- R5: renamed from J4; value RFID_ANT -> 10k; footprint Connector_Molex:Molex_PicoBlade_53047-0210_1x02_P1.25mm_Vertical -> Resistor_SMD:R_0603_1608Metric; symbol Connector_Generic:Conn_01x02 -> Device:R; MPN Molex 53047-0210 -> (none)
- R8: renamed from C5; value 1000uF 10V -> 1R; footprint Capacitor_SMD:CP_Elec_8x10.5 -> Resistor_SMD:R_0805_2012Metric; symbol Device:C_Polarized -> Device:R; LCSC C278408 -> (none); MPN Panasonic EEE-FT1A102AP -> (none)
- R9: renamed from C7; value 1000uF 10V -> 1R; footprint Capacitor_SMD:CP_Elec_8x10.5 -> Resistor_SMD:R_0805_2012Metric; symbol Device:C_Polarized -> Device:R; LCSC C278408 -> (none); MPN Panasonic EEE-FT1A102AP -> (none)
Connections:
- net +3V0: now also C4.1; no longer H1.1
- net +5V: now also R6.1; no longer C5.1
- net ANT1: now also J4.1 (Pin_1); no longer R5.1 (Pin_1)
- net ANT2: now also J4.2 (Pin_2); no longer R5.2 (Pin_2)
- net GND: now also C5.2, C4.2, C7.2, C8.2; no longer H1.2, R8.2, R9.2
- net RFID_TX_5V: now also R5.2
- net VCC_RF: now also R5.1, R9.2, C8.1
- net VRF1: now also C5.1, R6.2; no longer C5.2
- net VRF2: now also R8.2, C7.1
Other:
- note added: "CHG_INT: BQ25798 /INT is open-drain; pull-up is on the charger board (or enable the T4 GPIO1_A0 internal pull-up)"
- note removed: "R3: CHG_INT pull-up (BQ25798 /INT is open-drain)"
