File: lis3dh_board.kicad_pcb (KiCad board)
At the start: 2 copper layers, 102.9 x 25.4 mm, 26 parts, among them J1 T4_IF, J2 BQ25798_BOARD, J3 WL-125, J4 RFID_ANT, Q1 BSS138, U1 TLV75530PDBV, U2 LIS3DH

Commit message: Route the PCB and remove R3
- Remove R3 (CHG_INT pull-up); the pull-up lives on the charger board.
- Route the user's placement with Freerouting: netclasses Default
  (0.25mm), Power (+5V/VRF1/VRF2/VCC_RF, 0.4mm) and ANT (0.3mm, 0.4mm
  clearance), B.Cu GND plane, F.Cu GND pour plus 6 stitching vias.
  KiCad 10 DRC: no errors, 0 unconnected, schematic parity clean.
- Export Gerbers, drill and position files; add scripts/route.sh and
  route_pcb.py for re-routing; drop the obsolete gen_pcb.py.

Co-Authored-By: Claude Opus 5.5 <noreply@anthropic.com>
Claude-Session: https://claude.ai/code/session_012K15v8QNdkAoa4NiCNiWuG
Parts:
- removed R3: 10k, Resistor_SMD:R_0603_1608Metric
Routing:
- net /SCL: track 0.00 -> 100.4 mm
- net /SDA: track 0.00 -> 99.1 mm
- net +3V0: track 0.00 -> 97.5 mm
- net /INT1: track 0.00 -> 78.8 mm, vias 0 -> 1
- net /RFID_TX: track 0.00 -> 76.5 mm
- net /VCC_RF: track 0.00 -> 41.4 mm
- net /ANT2: track 0.00 -> 23.7 mm
- net /ANT1: track 0.00 -> 20.7 mm
- net /CHG_INT: track 0.00 -> 19.3 mm
- net +5V: track 0.00 -> 19.0 mm
- net GND: track 0.00 -> 16.6 mm, vias 0 -> 16
- net /VRF1: track 0.00 -> 13.9 mm
- net /VRF2: track 0.00 -> 13.6 mm
- net /RFID_TX_5V: track 0.00 -> 13.4 mm
- net /RFID_RST: track 0.00 -> 2.98 mm
- added copper zone on B.Cu, net GND
- added copper zone on F.Cu, net GND
