File: lis3dh_board.kicad_pcb (KiCad board)
At the start: 2 copper layers, 87.6 x 25.4 mm, 25 parts, among them J1 T4_IF, J2 BQ25798_BOARD, J3 WL-125, J4 RFID_ANT, Q1 BSS138, U1 TLV75530PDBV, U2 LIS3DH

Commit message: Route rfid_tx
Routing:
- net /RFID_TX: track 2.29 -> 57.7 mm, vias 0 -> 1
- net GND: vias 65 -> 70
Changed lines of the file:
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@@
+	)
+	(via
+		(at 116.332 95.758)
+		(size 0.6)
+		(drill 0.3)
+		(layers "F.Cu" "B.Cu")
+		(free yes)
+		(net "GND")
 	)
 	(via
@@
 	)
 	(via
+		(at 117.475 95.758)
+		(size 0.6)
+		(drill 0.3)
+		(layers "F.Cu" "B.Cu")
+		(free yes)
+		(net "GND")
+	)
+	(via
 		(at 160.528 91.694)
 		(size 0.6)
@@
 	)
 	(via
+		(at 114.681 98.679)
+		(size 0.6)
+		(drill 0.3)
+		(layers "F.Cu" "B.Cu")
+		(free yes)
+		(net "GND")
+	)
+	(via
 		(at 119.38 93.726)
 		(size 0.6)
@@
 	(via
 		(at 108.966 84.582)
+		(size 0.6)
+		(drill 0.3)
+		(layers "F.Cu" "B.Cu")
+		(free yes)
+		(net "GND")
+	)
+	(via
+		(at 120.396 95.758)
+		(size 0.6)
+		(drill 0.3)
+		(layers "F.Cu" "B.Cu")
+		(free yes)
+		(net "GND")
+	)
+	(via
+		(at 121.793 88.9)
 		(size 0.6)
 		(drill 0.3)
@@
 	)
 	(segment
+		(start 128.651 91.44)
+		(end 128.651 89.2635)
+		(width 0.25)
+		(layer "F.Cu")
+		(net "/RFID_TX")
+	)
+	(segment
+		(start 128.651 89.2635)
+		(end 128.6025 89.215)
+		(width 0.25)
+		(layer "F.Cu")
+		(net "/RFID_TX")
+	)
+	(segment
 		(start 128.6025 89.215)
 		(end 126.49 89.215)
@@
 		(net "/RFID_TX")
 	)
+	(via
+		(at 128.651 91.44)
+		(size 0.6)
+		(drill 0.3)
+		(layers "F.Cu" "B.Cu")
+		(net "/RFID_TX")
+	)
+	(segment
+		(start 128.651 91.44)
+		(end 133.731 96.52)
+		(width 0.25)
+		(layer "B.Cu")
+		(net "/RFID_TX")
+	)
+	(segment
+		(start 133.731 96.52)
+		(end 179.705 96.52)
+		(width 0.25)
+		(layer "B.Cu")
+		(net "/RFID_TX")
+	)
